File: usb-to-uart-bridge.kicad_sch (KiCad schematic)
At the start: 10 parts, among them J1 USB_C_Receptacle_USB2.0_16P, J2 Conn_01x05_Pin, U1 CP2102N-Axx-xQFN28

Commit message: Updated Schematic and Layout with CC Resistors
Parts:
- added R1, R2: 5.1K, Resistor_SMD:R_0402_1005Metric_Pad0.72x0.64mm_HandSolder, symbol Device:R
- U1: value CP2102N-Axx-xQFN28 -> CP2102N
Connections:
- net GND: now also R1.2, R2.2
- net at J1.A5 (CC1): now also R1.1
- net at J1.B5 (CC2): now also R2.1
- no-connect marks 23 -> 21
Other:
- note added: "Output Header"
- note added: "USB-C Connector"
- note added: "USB-to-UART Bridge Converter Breakout Module"
- note added: "USB-to-UART bridge controller"
- company: (none) -> HTronics
- title: (none) -> CP2102 USB To UART Bridge
